File: pcb/CanPressure.sch (KiCad schematic (older format))
At the start: 26 parts, among them IC101 ATTINY3224-SS, P102 CONN_5, P103 CAN, Q101 BSS138, Q102 BSS138, U101 MCP2515, U102 TJA1050, U103 NCP1117ST50T3G, U104 662K, U105 BMP280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

Commit message: Working in test harness  with a MCP2515 module
Connections:
- net MISO: now also IC101.12 ((RX1/MISO/AIN2)PA2); no longer IC101.11 ((TX1/MOSI/AIN1)PA1)
- net MOSI: now also IC101.11 ((TX1/MOSI/AIN1)PA1); no longer IC101.12 ((RX1/MISO/AIN2)PA2)
Changed lines of the file:
@@
 Text GLabel 5600 3900 2    60   Output ~ 0
 SCK
-Text GLabel 5600 4050 2    60   Output ~ 0
+Text GLabel 5600 4200 2    60   Output ~ 0
 MOSI
-Text GLabel 5600 4200 2    60   Input ~ 0
+Text GLabel 5600 4050 2    60   Input ~ 0
 MISO
 Text GLabel 3500 4050 0    60   Output ~ 0
